File: hardware/SolderOtto/_autosave-channel.kicad_sch (KiCad schematic)
At the start: 16 parts, among them J601 Conn_01x07

Commit message: save wip
Changed lines of the file:
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@@
 	)
 	(symbol
+		(lib_name "BAT54SFILM_1")
 		(lib_id "mylib_diodes:BAT54SFILM")
 		(at 43.18 175.26 90)
@@
 					(size 1.27 1.27)
 				)
+				(hide yes)
 			)
 		)
@@
 					(size 1.27 1.27)
 				)
+				(hide yes)
 			)
 		)
@@
 					(size 1.27 1.27)
 				)
+				(hide yes)
 			)
 		)
@@
 					(size 1.27 1.27)
 				)
-			)
-		)
+				(hide yes)
+			)
+		)
