File: hardware/SolderOtto/SolderOtto.kicad_pcb (KiCad board)
At the start: 4 copper layers, 165 x 70 mm, 0 parts

Commit message: create adapter to enclosure for display
Parts:
- added BT201: Battery_Cell, Battery:BatteryHolder_LINX_BAT-HLD-012-SMT, F.Cu at (252.0, 73.8)
- added C201: 3n3, Capacitor_SMD:C_0603_1608Metric, F.Cu at (-110.8, 52.8)
- added C202: 2n2, Capacitor_SMD:C_0603_1608Metric, F.Cu at (-110.8, 55.3)
- added C203: 47u, Capacitor_SMD:CP_Elec_10x10, F.Cu at (-105.5, 80.0)
- added C204: 2u2, Capacitor_SMD:C_1206_3216Metric, F.Cu at (-68.5, 95.0)
- added C205: 2u2, Capacitor_SMD:C_1206_3216Metric, F.Cu at (-68.5, 98.3)
- added C206: 47u, Capacitor_SMD:CP_Elec_10x10, F.Cu at (-105.5, 91.9)
- added C207: 56p, Capacitor_SMD:C_0603_1608Metric, F.Cu at (-110.8, 57.8)
- added C208: 10n, Capacitor_SMD:C_0603_1608Metric, F.Cu at (-110.8, 60.3)
- added C209: 10n, Capacitor_SMD:C_0603_1608Metric, F.Cu at (-110.8, 62.8)
- added C210: 10n, Capacitor_SMD:C_0603_1608Metric, F.Cu at (-110.8, 65.3)
- added C211: 10u, Capacitor_SMD:C_0805_2012Metric, F.Cu at (-79.1, 78.7)
- added C212: 10u, Capacitor_SMD:C_0805_2012Metric, F.Cu at (-79.1, 81.7)
- added C213: 10u, Capacitor_SMD:C_0805_2012Metric, F.Cu at (-79.1, 84.7)
- added C214: 22u, Capacitor_SMD:C_0805_2012Metric, F.Cu at (-79.1, 87.7)
- added C215: 22u, Capacitor_SMD:C_0805_2012Metric, F.Cu at (-79.1, 90.7)
- added C216: 22u, Capacitor_SMD:C_0805_2012Metric, F.Cu at (-79.1, 93.7)
- added C217: 4u7, Capacitor_SMD:C_0603_1608Metric, F.Cu at (-110.8, 67.8)
- added C218: 1u, Capacitor_SMD:C_0603_1608Metric, F.Cu at (-110.8, 70.3)
- added C219: 10u, Capacitor_SMD:C_0805_2012Metric, F.Cu at (-79.1, 96.7)
- added C220: 4u7, Capacitor_SMD:C_0603_1608Metric, F.Cu at (-110.8, 72.8)
- added C221: 1u, Capacitor_SMD:C_0603_1608Metric, F.Cu at (-106.8, 52.8)
- added C301: 100n, Resistor_SMD:R_0402_1005Metric, F.Cu at (191.6, 71.2)
- added C302: 100n, Resistor_SMD:R_0402_1005Metric, F.Cu at (187.6, 79.6)
- added C303: 100n, Resistor_SMD:R_0402_1005Metric, F.Cu at (187.6, 86.8)
- added C304: 100n, Resistor_SMD:R_0402_1005Metric, F.Cu at (198.1, 91.7)
- added C305: 100n, Resistor_SMD:R_0402_1005Metric, F.Cu at (203.6, 91.2)
- added C306: 100n, Resistor_SMD:R_0402_1005Metric, F.Cu at (207.6, 82.0)
- added C307: 100n, Resistor_SMD:R_0402_1005Metric, F.Cu at (207.6, 75.6)
- added C308: 100n, Resistor_SMD:R_0402_1005Metric, F.Cu at (198.4, 71.2)
- added C309: 4u7, Resistor_SMD:R_0402_1005Metric, F.Cu at (186.6, 79.6)
- added C310: 100n, Resistor_SMD:R_0402_1005Metric, F.Cu at (187.6, 77.2)
- added C311: 10n, Resistor_SMD:R_0402_1005Metric, F.Cu at (194.6, 91.2)
- added C312: 1u, Resistor_SMD:R_0402_1005Metric, F.Cu at (194.6, 92.2)
- added C313: 1u, Resistor_SMD:R_0402_1005Metric, F.Cu at (196.6, 91.2)
- added C314: 100n, Resistor_SMD:R_0402_1005Metric, F.Cu at (196.6, 92.2)
- added C315: 9p, Capacitor_SMD:C_0603_1608Metric, F.Cu at (-41.9, 104.8)
- added C316: 9p, Capacitor_SMD:C_0603_1608Metric, F.Cu at (-41.9, 107.3)
- added C317: 100n, Resistor_SMD:R_0402_1005Metric, F.Cu at (187.6, 82.8)
- added C601: 100n, Capacitor_SMD:C_0603_1608Metric, F.Cu at (-77.5, 111.1)
- added C602: 100n, Capacitor_SMD:C_0603_1608Metric, F.Cu at (-77.5, 113.6)
- added C603: 100n, Capacitor_SMD:C_0603_1608Metric, F.Cu at (-77.5, 116.1)
- added C604: 100n, Capacitor_SMD:C_0603_1608Metric, F.Cu at (-77.5, 118.6)
- added C801: 47p, Capacitor_SMD:C_0603_1608Metric, F.Cu at (-39.6, 52.8)
- added C802: 1n, Capacitor_SMD:C_0603_1608Metric, F.Cu at (-39.6, 55.3)
- added C803: 1u, Capacitor_SMD:C_0603_1608Metric, F.Cu at (-39.6, 57.8)
- added C804: 1u, Capacitor_SMD:C_0603_1608Metric, F.Cu at (-39.6, 60.3)
- added C805: 1u, Capacitor_SMD:C_0603_1608Metric, F.Cu at (-39.6, 62.8)
- added C806: 47p, Capacitor_SMD:C_0603_1608Metric, F.Cu at (-39.6, 67.8)
- added C807: 100p, Capacitor_SMD:C_0603_1608Metric, F.Cu at (-35.6, 52.8)
- added C808: 1u, Capacitor_SMD:C_0603_1608Metric, F.Cu at (-39.6, 65.3)
- added C809: 47p, Capacitor_SMD:C_0603_1608Metric, F.Cu at (-39.6, 70.3)
- added C810: 1n, Capacitor_SMD:C_0603_1608Metric, F.Cu at (-39.6, 72.8)
- added C811: 1u, Capacitor_SMD:C_0603_1608Metric, F.Cu at (-39.6, 75.4)
- added D201: STPS2H100A, Diode_SMD:D_SMA, F.Cu at (-61.6, 95.6)
- added D202: B380B-13-F, Diode_SMD:D_SMB, F.Cu at (-64.8, 68.8)
- added D203: SMD16PL-TP, Diode_SMD:D_SOD-123F, F.Cu at (-71.7, 67.7)
- added D204: SMD16PL-TP, Diode_SMD:D_SOD-123F, F.Cu at (-71.7, 71.1)
- added D205: SMD16PL-TP, Diode_SMD:D_SOD-123F, F.Cu at (-71.7, 74.4)
- added D206: BAT54SFILM, Package_TO_SOT_SMD:SOT-23, F.Cu at (-89.0, 68.5)
- added D207: BAT54SFILM, Package_TO_SOT_SMD:SOT-23, F.Cu at (213.4, 96.0)
- added D603: BAS70S, Package_TO_SOT_SMD:SOT-23, F.Cu at (-82.0, 112.2)
- added D604: BAT54SFILM, Package_TO_SOT_SMD:SOT-23, F.Cu at (-82.0, 116.9)
- added D605: BAT54SFILM, Package_TO_SOT_SMD:SOT-23, F.Cu at (-82.0, 121.5)
- added D606: BAT54SFILM, Package_TO_SOT_SMD:SOT-23, F.Cu at (-82.0, 126.1)
- added D801: BAT54SFILM, Package_TO_SOT_SMD:SOT-23, F.Cu at (-52.5, 53.9)
- added D802: BAT54SFILM, Package_TO_SOT_SMD:SOT-23, F.Cu at (-52.5, 58.5)
- added D803: BAT54SFILM, Package_TO_SOT_SMD:SOT-23, F.Cu at (-52.5, 63.2)
- added F801: 1.25A, Fuse:Fuse_0603_1608Metric, F.Cu at (-35.6, 55.3)
- added J201: Conn_02x04_Counter_Clockwise, Connector_Molex:Molex_Mini-Fit_Jr_5566-08A_2x04_P4.20mm_Vertical, F.Cu at (205.8, 120.3)
- added J301: TC-2050, mylib_connector:TC-2050, F.Cu at (166.3, 67.4)
- added J401: Conn_01x20, mylib_connector:FPC_BOTTOM_20POS_Würth_68712014522, F.Cu at (189.8, 63.0)
- added J501: Conn_01x08, Connector_Molex:Molex_Nano-Fit_105310-xx08_2x04_P2.50mm_Vertical, F.Cu at (217.3, 65.2)
- added J601: Conn_01x07, Connector_Molex:Molex_Micro-Fit_3.0_43650-0715_1x07_P3.00mm_Vertical, F.Cu at (-80.1, 105.5)
- added JS201: SMI-1027-T-5V-R, mylib_ic:SMI-1027-T-5V-R, F.Cu at (-80.5, 71.6)
- added L201: 33u, Inductor_SMD:L_Taiyo-Yuden_NR-80xx, F.Cu at (-66.6, 81.9)
- added L202: 1u5, Inductor_SMD:L_Taiyo-Yuden_NR-40xx, F.Cu at (-74.1, 79.9)
- added L203: 3u3, Inductor_SMD:L_Taiyo-Yuden_NR-40xx, F.Cu at (-74.1, 85.5)
- added L204: 3u3, Inductor_SMD:L_Taiyo-Yuden_NR-40xx, F.Cu at (-74.1, 91.0)
- added L301: 600R@100MHz, Inductor_SMD:L_0402_1005Metric, F.Cu at (194.6, 93.2)
- added P301: USB_C_Plug_USB2.0, mylib_connector:USB_C_Receptacle_Molex_C_24P_SMD_RA, F.Cu at (223.0, 90.0)
- added Q201: T2N7002AK, Package_TO_SOT_SMD:SOT-23, F.Cu at (-89.0, 77.7)
- added Q202: BC858B, Package_TO_SOT_SMD:SOT-23, F.Cu at (224.4, 111.1)
- added Q203: BC847A, Package_TO_SOT_SMD:SOT-23, F.Cu at (220.8, 115.1)
- added Q204: BC847A, Package_TO_SOT_SMD:SOT-23, F.Cu at (220.8, 111.1)
- added Q801: BC847A, Package_TO_SOT_SMD:SOT-23, F.Cu at (-52.5, 67.8)
- added Q802: BC858B, Package_TO_SOT_SMD:SOT-23, F.Cu at (-52.5, 72.4)
- added Q803: BC847A, Package_TO_SOT_SMD:SOT-23, F.Cu at (-52.5, 77.0)
- added Q901: Q_Dual_NMOS, Package_SO:SO-8_3.9x4.9mm_P1.27mm, F.Cu at (-108.6, 105.4)
- added Q902: Q_Dual_NMOS, Package_SO:SO-8_3.9x4.9mm_P1.27mm, F.Cu at (-108.6, 112.0)
- added Q903: Q_Dual_NMOS, Package_SO:SO-8_3.9x4.9mm_P1.27mm, F.Cu at (-108.6, 131.7)
- added Q904: DTD123EK, Package_TO_SOT_SMD:SC-59, F.Cu at (-92.9, 104.5)
- added Q905: DTD123EK, Package_TO_SOT_SMD:SC-59, F.Cu at (-92.9, 109.4)
- added Q906: DTD123EK, Package_TO_SOT_SMD:SC-59, F.Cu at (-92.9, 123.8)
- added Q907: Q_Dual_NMOS, Package_SO:SO-8_3.9x4.9mm_P1.27mm, F.Cu at (-108.6, 118.5)
- added Q908: Q_Dual_NMOS, Package_SO:SO-8_3.9x4.9mm_P1.27mm, F.Cu at (-108.6, 125.1)
- added Q909: DTD123EK, Package_TO_SOT_SMD:SC-59, F.Cu at (-92.9, 114.2)
- added Q910: DTD123EK, Package_TO_SOT_SMD:SC-59, F.Cu at (-92.9, 119.0)
- added R201: 453k, Resistor_SMD:R_0603_1608Metric, F.Cu at (-106.8, 55.3)
- added R202: 453k, Resistor_SMD:R_0603_1608Metric, F.Cu at (-106.8, 57.8)
- added R203: 100k, Resistor_SMD:R_0603_1608Metric, F.Cu at (-106.8, 60.3)
- added R204: 49k9, Resistor_SMD:R_0603_1608Metric, F.Cu at (-106.8, 62.8)
- added R205: 49k9, Resistor_SMD:R_0603_1608Metric, F.Cu at (-106.8, 65.3)
- added R206: 49k9, Resistor_SMD:R_0603_1608Metric, F.Cu at (-106.8, 67.8)
- added R207: 49k9, Resistor_SMD:R_0603_1608Metric, F.Cu at (-106.8, 70.3)
- added R208: 5k62, Resistor_SMD:R_0603_1608Metric, F.Cu at (-106.8, 72.8)
- added R209: 9k53, Resistor_SMD:R_0603_1608Metric, F.Cu at (-102.8, 52.8)
- added R210: 16k2, Resistor_SMD:R_0603_1608Metric, F.Cu at (-102.8, 55.3)
- added R211: 215k, Resistor_SMD:R_0603_1608Metric, F.Cu at (-102.8, 57.8)
- added R212: 4k7, Resistor_SMD:R_0603_1608Metric, F.Cu at (-102.8, 60.3)
- added R213: 69k, Resistor_SMD:R_0603_1608Metric, F.Cu at (-102.8, 62.8)
- added R214: 10k, Resistor_SMD:R_0603_1608Metric, F.Cu at (224.4, 114.0)
- added R215: 100, Resistor_SMD:R_0603_1608Metric, F.Cu at (-102.8, 67.8)
- added R216: 4k7, Resistor_SMD:R_0603_1608Metric, F.Cu at (-102.8, 70.3)
- added R217: 10k, Resistor_SMD:R_0603_1608Metric, F.Cu at (224.4, 115.8)
- added R218: 10k, Resistor_SMD:R_0603_1608Metric, F.Cu at (224.6, 107.6)
- added R219: 200, Resistor_SMD:R_0603_1608Metric, F.Cu at (-98.8, 55.3)
- added R220: 1M, Resistor_SMD:R_0603_1608Metric, F.Cu at (213.4, 100.6)
- added R221: 100k, Resistor_SMD:R_0603_1608Metric, F.Cu at (213.4, 99.0)
- added R222: 22k, Resistor_SMD:R_0603_1608Metric, F.Cu at (224.4, 118.0)
- added R223: 100k, Resistor_SMD:R_0603_1608Metric, F.Cu at (216.6, 99.0)
- added R224: 1M, Resistor_SMD:R_0603_1608Metric, F.Cu at (220.8, 118.0)
- added R301: 0, Resistor_SMD:R_0603_1608Metric, F.Cu at (219.2, 83.3)
- added R302: 0, Resistor_SMD:R_0603_1608Metric, F.Cu at (219.2, 86.0)
- added R303: 0, Resistor_SMD:R_0603_1608Metric, F.Cu at (227.0, 98.0)
- added R501: 4k7, Resistor_SMD:R_0603_1608Metric, F.Cu at (-47.6, 117.8)
- added R502: 4k7, Resistor_SMD:R_0603_1608Metric, F.Cu at (-47.6, 120.3)
- added R503: 4k7, Resistor_SMD:R_0603_1608Metric, F.Cu at (-47.6, 122.9)
- added R504: 4k7, Resistor_SMD:R_0603_1608Metric, F.Cu at (-47.6, 125.4)
- added R505: 4k7, Resistor_SMD:R_0603_1608Metric, F.Cu at (-47.6, 127.9)
- added R506: 4k7, Resistor_SMD:R_0603_1608Metric, F.Cu at (-47.6, 130.4)
- added R601: 4k7, Resistor_SMD:R_0603_1608Metric, F.Cu at (-77.5, 121.1)
- added R602: 4k7, Resistor_SMD:R_0603_1608Metric, F.Cu at (-77.5, 123.7)
- added R603: 4k7, Resistor_SMD:R_0603_1608Metric, F.Cu at (-73.5, 111.1)
- added R604: 4k7, Resistor_SMD:R_0603_1608Metric, F.Cu at (-73.5, 113.6)
- added R605: 4k7, Resistor_SMD:R_0603_1608Metric, F.Cu at (-73.5, 116.1)
- added R606: 4k7, Resistor_SMD:R_0603_1608Metric, F.Cu at (-73.5, 118.6)
- added R607: 4k7, Resistor_SMD:R_0603_1608Metric, F.Cu at (-73.5, 121.1)
- added R801: 82k, Resistor_SMD:R_0603_1608Metric, F.Cu at (-35.6, 57.8)
- added R802: 590k, Resistor_SMD:R_0603_1608Metric, F.Cu at (-35.6, 60.3)
- added R803: 22k6, Resistor_SMD:R_0603_1608Metric, F.Cu at (-35.6, 62.8)
- added R804: 22k6, Resistor_SMD:R_0603_1608Metric, F.Cu at (-35.6, 65.3)
- added R805: 2k7, Resistor_SMD:R_0603_1608Metric, F.Cu at (-35.6, 67.8)
- added R806: 20k, Resistor_SMD:R_0603_1608Metric, F.Cu at (-35.6, 70.3)
- added R807: 2k2, Resistor_SMD:R_0603_1608Metric, F.Cu at (-35.6, 72.8)
- added R808: 20k, Resistor_SMD:R_0603_1608Metric, F.Cu at (-35.6, 75.4)
- added R809: 2k55, Resistor_SMD:R_0603_1608Metric, F.Cu at (-23.6, 65.3)
- added R810: 22k6, Resistor_SMD:R_0603_1608Metric, F.Cu at (-23.6, 67.8)
- added R811: 22k6, Resistor_SMD:R_0603_1608Metric, F.Cu at (-31.6, 52.8)
- added R812: 590k, Resistor_SMD:R_0603_1608Metric, F.Cu at (-31.6, 55.3)
- added R813: 2k7, Resistor_SMD:R_0603_1608Metric, F.Cu at (-31.6, 57.8)
- added R814: 10k, Resistor_SMD:R_0603_1608Metric, F.Cu at (-23.6, 55.3)
- added R815: 200k, Resistor_SMD:R_0603_1608Metric, F.Cu at (-31.6, 60.3)
- added R816: 470k, Resistor_SMD:R_0603_1608Metric, F.Cu at (-23.6, 57.8)
- added R817: 47k, Resistor_SMD:R_0603_1608Metric, F.Cu at (-23.6, 60.3)
- added R818: 4k75, Resistor_SMD:R_0603_1608Metric, F.Cu at (-31.6, 62.8)
- added R819: 3k3, Resistor_SMD:R_0603_1608Metric, F.Cu at (-31.6, 65.3)
- added R820: 220m, Resistor_SMD:R_0603_1608Metric, F.Cu at (-31.6, 67.8)
- added R821: 10k, Resistor_SMD:R_0603_1608Metric, F.Cu at (-31.6, 70.3)
- added R822: 47k, Resistor_SMD:R_0603_1608Metric, F.Cu at (-23.6, 62.8)
- added R823: 3k3, Resistor_SMD:R_0603_1608Metric, F.Cu at (-31.6, 72.8)
- added R824: 220m, Resistor_SMD:R_0603_1608Metric, F.Cu at (-31.6, 75.4)
- added R825: 4k75, Resistor_SMD:R_0603_1608Metric, F.Cu at (-27.6, 52.8)
- added R826: 187k, Resistor_SMD:R_0603_1608Metric, F.Cu at (-27.6, 55.3)
- added R827: 1M, Resistor_SMD:R_0603_1608Metric, F.Cu at (-27.6, 60.3)
- added R828: 200k, Resistor_SMD:R_0603_1608Metric, F.Cu at (-27.6, 62.8)
- added R829: 10k, Resistor_SMD:R_0603_1608Metric, F.Cu at (-27.6, 65.3)
- added R830: 453k, Resistor_SMD:R_0603_1608Metric, F.Cu at (-27.6, 57.8)
- added R831: 3k3, Resistor_SMD:R_0603_1608Metric, F.Cu at (-27.6, 67.8)
- added R832: 20k, Resistor_SMD:R_0603_1608Metric, F.Cu at (-27.6, 70.3)
- added R833: 5m, Resistor_SMD:R_Shunt_Vishay_WSKW0612, F.Cu at (-30.0, 78.8)
- added R834: 3k3, Resistor_SMD:R_0603_1608Metric, F.Cu at (-27.6, 72.8)
- added R835: 20k, Resistor_SMD:R_0603_1608Metric, F.Cu at (-27.6, 75.4)
- added R836: 453k, Resistor_SMD:R_0603_1608Metric, F.Cu at (-23.6, 52.8)
- added R901: 470, Resistor_SMD:R_0603_1608Metric, F.Cu at (-88.4, 103.3)
- added R902: 470, Resistor_SMD:R_0603_1608Metric, F.Cu at (-88.4, 105.8)
- added R903: 470, Resistor_SMD:R_0603_1608Metric, F.Cu at (-88.4, 113.3)
- added R904: 470, Resistor_SMD:R_0603_1608Metric, F.Cu at (-88.4, 108.3)
- added R905: 470, Resistor_SMD:R_0603_1608Metric, F.Cu at (-88.4, 110.8)
- added REF**: MountingHole_3.2mm_M3, MountingHole:MountingHole_3.2mm_M3, F.Cu at (65.4, 125.0)
- added REF**: MountingHole_3.2mm_M3, MountingHole:MountingHole_3.2mm_M3, F.Cu at (225.0, 125.0)
- added REF**: MountingHole_3.2mm_M3, MountingHole:MountingHole_3.2mm_M3, F.Cu at (225.0, 55.0)
- added REF**: MountingHole_3.2mm_M3, MountingHole:MountingHole_3.2mm_M3, F.Cu at (65.4, 55.0)
- added SW301: SW_Push, Button_Switch_SMD:SW_Push_SPST_NO_Alps_SKRK, F.Cu at (170.0, 61.0)
- added TP201: ZCD, TestPoint:TestPoint_Keystone_5019_Minature, F.Cu at (211.2, 127.0)
- added TP202: ZCD, TestPoint:TestPoint_Keystone_5015_Micro-Minature, F.Cu at (220.9, 107.6)
- added TP203: ZCD, TestPoint:TestPoint_Keystone_5015_Micro-Minature, F.Cu at (216.8, 96.0)
- added TP501: ZCD, TestPoint:TestPoint_Keystone_5015_Micro-Minature, F.Cu at (-52.3, 137.2)
- added TP502: ZCD, TestPoint:TestPoint_Keystone_5015_Micro-Minature, F.Cu at (-52.3, 122.2)
- added TP503: ZCD, TestPoint:TestPoint_Keystone_5015_Micro-Minature, F.Cu at (-52.3, 118.5)
- added TP504: ZCD, TestPoint:TestPoint_Keystone_5015_Micro-Minature, F.Cu at (-52.3, 126.0)
- added TP505: ZCD, TestPoint:TestPoint_Keystone_5015_Micro-Minature, F.Cu at (-52.3, 129.7)
- added TP506: ZCD, TestPoint:TestPoint_Keystone_5015_Micro-Minature, F.Cu at (-52.3, 133.5)
- added TP801: T_TIP, TestPoint:TestPoint_Keystone_5015_Micro-Minature, F.Cu at (-18.9, 53.4)
- added TP802: DET, TestPoint:TestPoint_Keystone_5015_Micro-Minature, F.Cu at (-18.9, 64.6)
- added TP803: I_LEAK, TestPoint:TestPoint_Keystone_5015_Micro-Minature, F.Cu at (-18.9, 57.1)
- added TP804: I_LOAD, TestPoint:TestPoint_Keystone_5015_Micro-Minature, F.Cu at (-18.9, 60.9)
- added U201: LM5012, Package_SO:TI_SO-PowerPAD-8, F.Cu at (-66.8, 90.1)
- added U202: AP3211K, Package_TO_SOT_SMD:SOT-23-6, F.Cu at (-83.9, 79.6)
- added U203: AP3211K, Package_TO_SOT_SMD:SOT-23-6, F.Cu at (-83.9, 84.2)
- added U204: AP3211K, Package_TO_SOT_SMD:SOT-23-6, F.Cu at (-83.9, 88.8)
- added U205: LM27761, Package_SON:WSON-8-1EP_2x2mm_P0.5mm_EP0.9x1.6mm, F.Cu at (-66.8, 73.5)
- added U206: MCP9701T-E/TT, Package_TO_SOT_SMD:SOT-23-3, F.Cu at (-83.9, 93.4)
- added U301: USBLC6-2SC6, Package_TO_SOT_SMD:SOT-23-6, F.Cu at (219.0, 90.0)
- added U302: STM32G474QETx, Package_QFP:LQFP-128_14x14mm_P0.4mm, F.Cu at (197.6, 81.2)
- added U303: MX25R3235FM1xx0, Package_SO:SOP-8_3.9x4.9mm_P1.27mm, F.Cu at (191.4, 105.1)
- added U701: SN74LVC125A, Package_SO:TSSOP-14_4.4x5mm_P0.65mm, F.Cu at (-28.3, 119.9)
- added U702: TS5A3159ADCK, Package_TO_SOT_SMD:SOT-363_SC-70-6, F.Cu at (-30.6, 125.2)
- added U801: OP07, Package_SO:SOIC-8_3.9x4.9mm_P1.27mm, F.Cu at (-45.8, 54.9)
- added U802: LM358, Package_SO:SOIC-8_3.9x4.9mm_P1.27mm, F.Cu at (-45.8, 61.5)
- added U803: 74hc4053, Package_SO:TSSOP-16_4.4x5mm_P0.65mm, F.Cu at (-36.9, 79.9)
- added U804: OP07, Package_SO:SOIC-8_3.9x4.9mm_P1.27mm, F.Cu at (-45.8, 68.0)
- added U805: OP07, Package_SO:SOIC-8_3.9x4.9mm_P1.27mm, F.Cu at (-45.8, 74.6)
- added U901: VOM1271, mylib_ic:SOP-4_3.8x4.1mm_P2.54mm, F.Cu at (-99.8, 105.0)
- added U902: VOM1271, mylib_ic:SOP-4_3.8x4.1mm_P2.54mm, F.Cu at (-99.8, 110.8)
- added U903: VOM1271, mylib_ic:SOP-4_3.8x4.1mm_P2.54mm, F.Cu at (-99.8, 128.3)
- added U904: VOM1271, mylib_ic:SOP-4_3.8x4.1mm_P2.54mm, F.Cu at (-99.8, 116.7)
- added U905: VOM1271, mylib_ic:SOP-4_3.8x4.1mm_P2.54mm, F.Cu at (-99.8, 122.5)
- added Y301: 32.768 kHz, Crystal:Crystal_SMD_MicroCrystal_CC8V-T1A-2Pin_2.0x1.2mm, F.Cu at (-29.5, 109.7)
Routing:
- net Net-(Q203-E): track 0.00 -> 5.88 mm
- net GND: track 0.00 -> 5.88 mm
- net Net-(Q202-B): track 0.00 -> 3.85 mm
- net /Supply/ZCD: track 0.00 -> 2.78 mm
- net Net-(Q203-C): track 0.00 -> 2.12 mm
- net +3V3: track 0.00 -> 2.05 mm
Other:
- board size 165 x 70 mm -> 169.6 x 80 mm

Commit message: save work
Parts:
- removed BT201: Battery_Cell, Battery:BatteryHolder_LINX_BAT-HLD-012-SMT
- removed the REF** at (65.4, 125.0)
- removed the REF** at (225.0, 125.0)
- removed the REF** at (225.0, 55.0)
- removed the REF** at (65.4, 55.0)
- added C315: 100n, Capacitor_SMD:C_0603_1608Metric, F.Cu at (211.3, 108.7)
- added C319: 10n, Capacitor_SMD:C_0603_1608Metric, F.Cu at (226.0, 98.4)
- added REF**: MountingHole_2.2mm_M2, MountingHole:MountingHole_2.2mm_M2, F.Cu at (226.0, 128.0)
- added TP201: 24V~, TestPoint:TestPoint_Keystone_5015_Micro-Minature, F.Cu at (225.8, 116.3)
- added TP202: 12V, TestPoint:TestPoint_Keystone_5015_Micro-Minature, F.Cu at (189.3, 126.0)
- added TP204: 8V, TestPoint:TestPoint_Keystone_5015_Micro-Minature, F.Cu at (174.6, 101.8)
- added TP205: 5V, TestPoint:TestPoint_Keystone_5015_Micro-Minature, F.Cu at (174.6, 120.8)
- added TP206: 3V3, TestPoint:TestPoint_Keystone_5015_Micro-Minature, F.Cu at (174.6, 90.3)
- C203, C206: value 47u -> 22u; footprint Capacitor_SMD:CP_Elec_10x10 -> Capacitor_SMD:CP_Elec_6.3x5.7
- C316: renamed from C315; footprint Capacitor_SMD:C_0603_1608Metric -> Capacitor_SMD:C_0402_1005Metric
- C317: renamed from C316; footprint Capacitor_SMD:C_0603_1608Metric -> Capacitor_SMD:C_0402_1005Metric
- R303: value 0 -> 1M
- TP203: renamed from TP201; value ZCD -> GND
- TP208: renamed from TP203; value ZCD -> V_{ANA}
- TP501: value ZCD -> EXT0
- TP502: value ZCD -> EXT1
- TP503: value ZCD -> EXT2
- TP504: value ZCD -> EXT3
- TP505: value ZCD -> EXT4
- TP506: value ZCD -> EXT5
- TP901: renamed from TP801; value T_TIP -> T_{TIP}
- TP903: renamed from TP803; value I_LEAK -> I_{LEAK}
- TP904: renamed from TP804; value I_LOAD -> I_{LOAD}
- U303: footprint Package_SO:SOP-8_3.9x4.9mm_P1.27mm -> Package_SO:SOIC-8_3.9x4.9mm_P1.27mm
- moved C221 324.2 mm to (214.4, 97.1), turned to 180 degrees
- moved C203 321.1 mm to (212.3, 125.6), turned to -90 degrees
- moved R219 320.0 mm to (217.9, 100.9), turned to 180 degrees
- moved R203 317.7 mm to (206.2, 115.0), turned to 180 degrees
- moved C202 315.7 mm to (198.2, 119.9), turned to 90 degrees
- moved C207 314.6 mm to (198.2, 116.8), turned to 90 degrees
- moved C201 314.0 mm to (196.6, 116.8), turned to 90 degrees
- moved R204 313.4 mm to (202.3, 115.0)
- moved R212 311.2 mm to (208.2, 73.0), turned to -90 degrees
- moved R201 310.2 mm to (196.6, 119.9), turned to -90 degrees
- moved R202 309.4 mm to (197.4, 114.5)
- moved D206 305.2 mm to (214.6, 99.9), turned to 90 degrees
- moved U206 302.5 mm to (218.5, 98.0)
- moved R215 297.7 mm to (194.8, 76.6), turned to 180 degrees
- moved R216 297.6 mm to (194.8, 73.8)
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- renumbered C317 to C318, C801 to C901, C802 to C902, C803 to C903, C804 to C904, C805 to C905, C806 to C906, C807 to C907, C808 to C908, C809 to C909, C810 to C910, C811 to C911, D801 to D901, D802 to D902, D803 to D903, F801 to F901, Q901 to Q801, Q902 to Q802, Q903 to Q803, Q904 to Q804, Q905 to Q805, Q906 to Q806, Q907 to Q807, Q908 to Q808, Q909 to Q809, Q910 to Q810, Q801 to Q901, Q802 to Q902, Q803 to Q903, R901 to R801, R902 to R802, R903 to R803, R904 to R804, R905 to R805, R801 to R901, R802 to R902, R803 to R903, R804 to R904, R805 to R905, R806 to R906, R807 to R907, R808 to R908, R809 to R909, R810 to R910, R811 to R911, R812 to R912, R813 to R913, R814 to R914, R815 to R915, R816 to R916, R817 to R917, R818 to R918, R819 to R919, R820 to R920, R821 to R921, R822 to R922, R823 to R923, R824 to R924, R825 to R925, R826 to R926, R827 to R927, R828 to R928, R829 to R929, R830 to R930, R831 to R931, R832 to R932, R833 to R933, R834 to R934, R835 to R935, R836 to R936, TP202 to TP207, TP802 to TP902, U901 to U801, U902 to U802, U903 to U803, U904 to U804, U905 to U805, U801 to U901, U802 to U902, U803 to U903, U804 to U904, U805 to U905
Connections:
- C310 pad 1: VBAT -> +3V3
- J501 pad 5: /External connection/EXT_3 -> GND
- J501 pad 6: /External connection/EXT_4 -> /External connection/EXT_3
- J501 pad 7: /External connection/EXT_5 -> /External connection/EXT_4
- J501 pad 8: GND -> /External connection/EXT_5
- R303 pad 1: Earth -> Net-(P301-SHIELD)
- R303 pad 2: Net-(P301-SHIELD) -> Earth
- U302 pad 6: VBAT -> +3V3
Routing:
- net GND: track 5.88 -> 70.9 mm, vias 0 -> 4
- net +3V3: track 2.05 -> 42.5 mm
- net +12V: track 0.00 -> 34.5 mm
- net +5V: track 0.00 -> 21.1 mm, vias 0 -> 2
- net Net-(JS201--): track 0.00 -> 16.1 mm
- net /mcu/_D+: track 0.00 -> 14.8 mm, vias 0 -> 2
- net Net-(D201-K): track 0.00 -> 14.5 mm
- net Net-(D202-K): track 0.00 -> 13.6 mm
- net /mcu/_D-: track 0.00 -> 13.6 mm, vias 0 -> 2
- net /Supply/V_{ANA}: track 0.00 -> 10.5 mm
- net VDDA: track 0.00 -> 9.53 mm
- net 24V_{AC}: track 0.00 -> 9.37 mm
- net Net-(D205-K): track 0.00 -> 9.07 mm
- net Net-(D203-K): track 0.00 -> 9.07 mm
- net Net-(U905--): track 0.00 -> 9.07 mm
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- added copper zone on F.Cu, net +12V
- added copper zone on F.Cu, net +3V3
- added copper zone on F.Cu, net +5V
- added copper zone on F.Cu, net +8V
- added copper zone on F.Cu, net Net-(D201-K)
- added copper zone on F.Cu, net Net-(D202-K)
- added copper zone on F.Cu, net Net-(D203-K)
- added copper zone on F.Cu, net Net-(D204-K)
- added copper zone on F.Cu, net Net-(D205-K)
Other:
- board size 169.6 x 80 mm -> 169.6 x 84 mm

Commit message: save work
Parts:
- moved TP902 28.1 mm to (165.7, 124.0)
- moved R922 27.4 mm to (158.1, 123.5)
- moved Q903 27.2 mm to (161.6, 128.0)
- moved Q901 22.6 mm to (161.6, 124.4)
- moved Q902 22.0 mm to (165.4, 127.0), turned to 180 degrees
- moved R917 20.7 mm to (168.6, 127.0), turned to -90 degrees
- moved R916 19.6 mm to (158.8, 126.3), turned to 90 degrees
- moved R914 18.7 mm to (168.6, 124.0), turned to 90 degrees
- moved C907 17.9 mm to (158.1, 128.9), turned to 180 degrees
- moved D902 11.1 mm to (135.6, 125.3), turned to -90 degrees
- moved R905 8.43 mm to (118.6, 125.8)
- moved C903 8.43 mm to (121.8, 125.8)
- moved R902 8.43 mm to (123.7, 121.2)
- moved R912 8.43 mm to (116.7, 121.2)
- moved U901 8.43 mm to (120.2, 121.2)
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Routing:
- net Net-(U901-+): track 5.14 -> 17.3 mm
- net Net-(U901--): track 2.85 -> 13.2 mm
- net Net-(U903-3Y1): track 0.90 -> 9.07 mm, vias 1 -> 0
- net +3V3: track 42.5 -> 48.7 mm
- net Net-(U903-1Y1): track 0.00 -> 6.21 mm
- net /Channel0/_stand_sense: track 0.00 -> 3.35 mm
- net /Channel0/I_{LOAD}: track 0.00 -> 3.10 mm
- net /Channel0/stand_sense: track 0.00 -> 2.48 mm
- net /Channel0/DET: track 0.00 -> 2.38 mm
- net Net-(U902B--): track 0.00 -> 2.10 mm
- net Net-(R907-Pad1): track 0.00 -> 2.10 mm
- net Net-(R803-Pad2): track 0.00 -> 2.05 mm
- net Net-(R802-Pad2): track 0.00 -> 2.05 mm
- net Net-(R805-Pad2): track 0.00 -> 2.05 mm
- net Net-(Q806-C): track 0.00 -> 1.67 mm
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
Commit message: save work
Parts:
- removed REF**: MountingHole_2.2mm_M2, MountingHole:MountingHole_2.2mm_M2
- moved C219 66.4 mm to (116.1, 97.4), turned to 90 degrees
- moved C220 65.2 mm to (118.1, 97.2), turned to 90 degrees
- moved C217 64.2 mm to (119.6, 97.2), turned to 90 degrees
- moved R211 62.1 mm to (116.1, 101.0), turned to -90 degrees
- moved U205 60.1 mm to (118.8, 101.0), turned to -90 degrees
- moved R213 58.1 mm to (116.1, 104.5), turned to -90 degrees
- moved C218 56.4 mm to (119.3, 103.7), turned to 180 degrees
- moved R206 54.4 mm to (125.2, 104.3)
- moved TP205 54.4 mm to (125.2, 98.0)
- moved C209 54.4 mm to (130.2, 101.4)
- moved C212 54.4 mm to (133.6, 104.2)
- moved C215 54.4 mm to (126.2, 101.4)
- moved D203 54.4 mm to (133.6, 98.0)
- moved L203 54.4 mm to (130.0, 98.0)
- moved R209 54.4 mm to (127.1, 104.3)
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Connections:
- C901 pad 1: Net-(U901--) -> /Channel0/channel_meas/IN-
- R902 pad 1: Net-(U901--) -> /Channel0/channel_meas/IN-
- R903 pad 2: Net-(U903-3Y0) -> Net-(U903-1Y0)
- R904 pad 2: Net-(U903-3Y1) -> Net-(U903-1Y1)
- R906 pad 1: /Channel0/LOAD -> /Channel0/_iron_sense
- R906 pad 2: Net-(U903-2Y0) -> Net-(U903-3Y0)
- R908 pad 2: Net-(U903-2Y1) -> Net-(U903-3Y1)
- R909 pad 2: Net-(U903-1Y0) -> Net-(U903-2Y0)
- R910 pad 1: /Channel0/_iron_sense -> /Channel0/LOAD
- R910 pad 2: Net-(U903-1Y1) -> Net-(U903-2Y1)
- U901 pad 2: Net-(U901--) -> /Channel0/channel_meas/IN-
- U903 pad 11: /Channel0/SEL1 -> /Channel0/SEL3
- U903 pad 14: Net-(U901-+) -> /Channel0/channel_meas/IN-
- U903 pad 15: /Channel0/channel_meas/select -> Net-(U901-+)
- U903 pad 4: Net-(U901--) -> /Channel0/channel_meas/select
- U903 pad 9: /Channel0/SEL3 -> /Channel0/SEL1
Routing:
- net +12V: track 34.5 -> 77.0 mm, vias 0 -> 1
- net GND: track 70.9 -> 94.8 mm, vias 4 -> 7
- net /Channel0/TC: track 0.00 -> 20.9 mm
- net /Channel0/channel_meas/IN-: track 0.00 -> 20.6 mm
- net 24V_{AC}: track 9.37 -> 27.5 mm
- net /mcu/QSPI_IO2: track 2.99 -> 16.9 mm
- net /mcu/QSPI_IO1: track 2.45 -> 16.2 mm
- net Net-(U901--): track 13.2 -> 0.00 mm
- net /mcu/QSPI_CLK: track 2.41 -> 15.4 mm
- net /mcu/QSPI_IO0: track 6.87 -> 19.8 mm
- net /mcu/QSPI_NCS: track 8.42 -> 21.2 mm
- net /mcu/QSPI_IO3: track 2.27 -> 15.0 mm
- net /Channel0/channel_power/COM_SW_LOW: track 0.00 -> 10.6 mm, vias 0 -> 2
- net /mcu/_D+: track 14.8 -> 4.80 mm, vias 2 -> 0
- net /mcu/_D-: track 13.6 -> 4.80 mm, vias 2 -> 0
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Other:
- board size 169.6 x 84 mm -> 121 x 60 mm
