File: hardware/SolderOtto/SolderOtto_4_lay.kicad_pcb (KiCad board)
At the start: 2 copper layers, 125 x 60 mm, 232 parts, among them J201 Conn_02x04_Counter_Clockwise, J301 TC-2050, J401 Conn_01x20, J501 Conn_01x05, J601 Conn_01x07, P301 USB_C_Plug_USB2.0, Q201 T2N7002AK, Q202 BC858B, Q203 BC847A, Q204 BC847A, Q801 Q_Dual_NMOS, Q802 Q_Dual_NMOS, Q803 Q_Dual_NMOS, Q804 DTD123EK, Q805 DTD123EK, Q806 DTD123EK, Q807 Q_Dual_NMOS, Q808 Q_Dual_NMOS, Q809 DTD123EK, Q810 DTD123EK, SW301 SW_Push, U201 LM5012, U202 AP3211K, U203 AP3211K, U204 AP3211K, U205 LM27761, U206 MCP9701T-E/TT, U301 USBLC6-2SC6, U302 STM32G474QETx, U303 MX25R3235FM1xx0, U701 SN74LVC125A, U801 VOM1271, U802 VOM1271, U803 VOM1271, U804 VOM1271, U805 VOM1271, U901 OPA202, U902 LM358B, U903 74hc4053, U904 OPA202, U905 OPA202, U906 OPA202, U907 LM358B, U908 74hc4053, Y301 32.768 kHz

Commit message: rework pcb
Parts:
- C203, C206: value 100u -> 22u; footprint mylib_common:CP_Elec_10x10.5_A768 -> Capacitor_SMD:CP_Elec_10x10
- moved R215 16.9 mm to (226.6, 68.0), turned to -90 degrees
- moved R216 15.1 mm to (223.8, 68.0), turned to 90 degrees
- moved Q201 14.0 mm to (219.8, 68.0), turned to 180 degrees
- moved TP504 13.6 mm to (210.9, 63.4)
- moved TP503 7.19 mm to (207.7, 63.4)
- moved R212 7.04 mm to (219.8, 54.5), turned to 0 degrees
- moved TP501 6.11 mm to (201.2, 63.4)
- moved J501 4.05 mm to (210.2, 57.2)
- moved R501 4.05 mm to (210.1, 60.4)
- moved R502 4.05 mm to (206.8, 60.4)
- moved R503 4.05 mm to (203.6, 60.4)
- moved R504 4.05 mm to (200.3, 60.4)
- moved R917 1.93 mm to (112.9, 85.5)
- moved R919 1.93 mm to (110.8, 74.0)
- moved C910 1.93 mm to (110.0, 79.7)
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Connections:
- C903 pad 1: /Channel0/T_{TIP}_{a} -> /Channel0/channel_meas/T_{TIP}_{a}
- C917 pad 1: /Channel0/T_{TIP}_{b} -> /Channel0/channel_meas/T_{TIP}_{b}
- D901 pad 3: /Channel0/T_{TIP}_{a} -> /Channel0/channel_meas/T_{TIP}_{a}
- D904 pad 3: /Channel0/T_{TIP}_{b} -> /Channel0/channel_meas/T_{TIP}_{b}
- R906 pad 2: /Channel0/T_{TIP}_{a} -> /Channel0/channel_meas/T_{TIP}_{a}
- R935 pad 2: /Channel0/T_{TIP}_{b} -> /Channel0/channel_meas/T_{TIP}_{b}
- TP901 pad 1: /Channel0/T_{TIP}_{a} -> /Channel0/channel_meas/T_{TIP}_{a}
- TP904 pad 1: /Channel0/T_{TIP}_{b} -> /Channel0/channel_meas/T_{TIP}_{b}
- U302 pad 10: /Channel0/LOW_SIDE_COM -> unconnected-(U302-PF3-Pad10)
- U302 pad 100: /External connection/EXT_1 -> unconnected-(U302-PC10-Pad100)
- U302 pad 101: /External connection/EXT_2 -> unconnected-(U302-PC11-Pad101)
- U302 pad 102: /External connection/EXT_3 -> unconnected-(U302-PC12-Pad102)
- U302 pad 103: unconnected-(U302-PG5-Pad103) -> /Channel0/tip_change
- U302 pad 104: unconnected-(U302-PG6-Pad104) -> /mcu/Channel1_tip
- U302 pad 105: unconnected-(U302-PG7-Pad105) -> /mcu/Channel2_tip
- U302 pad 106: unconnected-(U302-PG8-Pad106) -> /mcu/Channel3_tip
- U302 pad 108: unconnected-(U302-PD0-Pad108) -> /Channel0/iron_sense
- U302 pad 11: /Channel0/LOAD1_SW -> unconnected-(U302-PF4-Pad11)
- U302 pad 112: unconnected-(U302-PD2-Pad112) -> /External connection/EXT_0
- U302 pad 113: unconnected-(U302-PD3-Pad113) -> /External connection/EXT_1
- U302 pad 114: unconnected-(U302-PD4-Pad114) -> /External connection/EXT_2
- U302 pad 115: unconnected-(U302-PD5-Pad115) -> /External connection/EXT_3
- U302 pad 119: unconnected-(U302-PB4-Pad119) -> /mcu/Channel1_iron
- U302 pad 120: unconnected-(U302-PB5-Pad120) -> /mcu/Channel2_iron
- U302 pad 122: unconnected-(U302-PB7-Pad122) -> /mcu/Channel3_iron
- U302 pad 125: unconnected-(U302-PE0-Pad125) -> /Supply/ZCD
- U302 pad 14: /Channel0/COM_SW -> unconnected-(U302-PF5-Pad14)
- U302 pad 15: /Channel0/LOW_SIDE_LOAD -> unconnected-(U302-PF7-Pad15)
- U302 pad 16: /Channel0/SEL1_{a} -> /Channel0/SEL1
- U302 pad 17: /Channel0/SEL1_{b} -> /Channel0/SEL2
- U302 pad 18: /Channel0/SEL2_{a} -> /Channel0/SEL3
- U302 pad 19: /Channel0/SEL2_{b} -> unconnected-(U302-PF0-Pad19)
- U302 pad 24: /Channel0/T_{TIP}_{a} -> /Channel0/T_{TIP}
- U302 pad 25: /Channel0/T_{TIP}_{b} -> /Channel0/I_{LEAK}
- U302 pad 26: unconnected-(U302-PF2-Pad26) -> /Channel0/LOW_SIDE_LOAD
- U302 pad 27: /Channel0/I_{LEAK} -> /Channel0/COM_SW
- U302 pad 28: unconnected-(U302-PA1-Pad28) -> /Channel0/LOAD0_SW
- U302 pad 29: unconnected-(U302-PA2-Pad29) -> /Channel0/LOAD1_SW
- U302 pad 32: unconnected-(U302-PA3-Pad32) -> /Channel0/LOW_SIDE_COM
- U302 pad 33: unconnected-(U302-PA4-Pad33) -> /mcu/Channel1_handle
- U302 pad 34: /Channel0/tip_change -> /mcu/Channel1_T_{TIP}
- U302 pad 35: /Channel0/stand_sense -> /mcu/Channel1_I_{LEAK}
- U302 pad 36: /Channel0/iron_sense -> /mcu/Channel1_I_{LOAD}
- U302 pad 38: unconnected-(U302-PC5-Pad38) -> /mcu/Channel1_LOW_SIDE_SW
- U302 pad 39: unconnected-(U302-PB0-Pad39) -> /mcu/Channel1_LOAD0_SW
- U302 pad 40: unconnected-(U302-PB1-Pad40) -> /mcu/Channel1_LOAD1_SW
- U302 pad 41: unconnected-(U302-PB2-Pad41) -> /mcu/Channel1_COM_SW
- U302 pad 48: unconnected-(U302-PF11-Pad48) -> /mcu/Channel1_SEL1
- U302 pad 49: unconnected-(U302-PF12-Pad49) -> /mcu/Channel1_SEL2
- U302 pad 50: unconnected-(U302-PF13-Pad50) -> /mcu/Channel1_SEL3
- U302 pad 52: unconnected-(U302-PF15-Pad52) -> /mcu/Channel2_SEL3
- U302 pad 53: unconnected-(U302-PE7-Pad53) -> /mcu/Channel2_I_{LEAK}
- U302 pad 54: unconnected-(U302-PE8-Pad54) -> /mcu/Channel2_T_{TIP}
- U302 pad 55: unconnected-(U302-PE9-Pad55) -> /mcu/Channel2_handle
- U302 pad 62: unconnected-(U302-PB10-Pad62) -> /mcu/Channel2_SEL1
- U302 pad 65: unconnected-(U302-PB11-Pad65) -> /mcu/Channel2_SEL2
- U302 pad 66: unconnected-(U302-PB12-Pad66) -> /Channel0/stand_sense
- U302 pad 67: unconnected-(U302-PB13-Pad67) -> /mcu/Channel1_stand
- U302 pad 68: unconnected-(U302-PB14-Pad68) -> /mcu/Channel2_stand
- U302 pad 69: unconnected-(U302-PB15-Pad69) -> /mcu/Channel3_stand
- U302 pad 7: /Channel0/LOAD0_SW -> /Supply/Buzzer
- U302 pad 72: unconnected-(U302-PD10-Pad72) -> /mcu/Channel2_I_{LOAD}
- U302 pad 73: unconnected-(U302-PD11-Pad73) -> /mcu/Channel3_I_{LOAD}
- U302 pad 74: unconnected-(U302-PD12-Pad74) -> /mcu/Channel3_I_{LEAK}
- U302 pad 75: unconnected-(U302-PD13-Pad75) -> /mcu/Channel3_T_{TIP}
- U302 pad 76: unconnected-(U302-PD14-Pad76) -> /mcu/Channel3_handle
- U302 pad 77: unconnected-(U302-PD15-Pad77) -> /mcu/Channel2_COM_SW
- U302 pad 80: unconnected-(U302-PC6-Pad80) -> /mcu/Channel2_LOAD0_SW
- U302 pad 81: unconnected-(U302-PC7-Pad81) -> /mcu/Channel2_LOAD1_SW
- U302 pad 82: unconnected-(U302-PG0-Pad82) -> /mcu/Channel2_LOW_SIDE_SW
- U302 pad 83: /Supply/ZCD -> /mcu/Channel3_SEL1
- U302 pad 84: unconnected-(U302-PG2-Pad84) -> /mcu/Channel3_SEL2
- U302 pad 85: unconnected-(U302-PG3-Pad85) -> /mcu/Channel3_SEL3
- U302 pad 86: unconnected-(U302-PG4-Pad86) -> /mcu/Channel3_COM_SW
- U302 pad 87: unconnected-(U302-PC8-Pad87) -> /mcu/Channel3_LOAD0_SW
- U302 pad 88: unconnected-(U302-PC9-Pad88) -> /mcu/Channel3_LOAD1_SW
- U302 pad 89: unconnected-(U302-PA8-Pad89) -> /mcu/Channel3_LOW_SIDE_SW
- U302 pad 97: /Supply/Buzzer -> unconnected-(U302-PF6-Pad97)
- U302 pad 99: /External connection/EXT_0 -> unconnected-(U302-PA15-Pad99)
- U701 pad 5: /Channel0/LOAD1_SW -> /Channel0/LOAD0_SW
- U701 pad 6: /Channel0/channel_power/LOAD1_SW_HIGH -> /Channel0/channel_power/LOAD0_SW_HIGH
- U701 pad 8: /Channel0/channel_power/LOAD0_SW_HIGH -> /Channel0/channel_power/LOAD1_SW_HIGH
- U701 pad 9: /Channel0/LOAD0_SW -> /Channel0/LOAD1_SW
- U903 pad 10: /Channel0/SEL1_{b} -> /Channel0/SEL2
- U903 pad 9: /Channel0/SEL1_{a} -> /Channel0/SEL1
- U907 pad 1: unconnected-(U907-Pad1) -> (no net)
- U907 pad 2: unconnected-(U907A---Pad2) -> (no net)
- U907 pad 3: unconnected-(U907A-+-Pad3) -> (no net)
- U908 pad 10: /Channel0/SEL2_{b} -> /Channel0/SEL2
- U908 pad 9: /Channel0/SEL2_{a} -> /Channel0/SEL1
Routing:
- net GND: track 716.3 -> 165.3 mm, vias 391 -> 41
- net +3V3: track 379.4 -> 58.0 mm, vias 39 -> 10
- net +5V: track 210.2 -> 21.1 mm, vias 6 -> 1
- net +12V: track 186.5 -> 20.7 mm, vias 8 -> 3
- net Earth: track 149.4 -> 3.01 mm, vias 4 -> 0
- net 24V_{AC}: track 147.5 -> 7.77 mm, vias 2 -> 0
- net +8V: track 134.5 -> 23.5 mm, vias 11 -> 0
- net /Channel0/I_{LEAK}: track 103.5 -> 0.00 mm
- net -5V: track 113.0 -> 27.1 mm, vias 9 -> 1
- net /Channel0/SEL1_{a}: track 81.7 -> 0.00 mm, vias 4 -> 0
- net /Channel0/SEL1_{b}: track 81.4 -> 0.00 mm, vias 4 -> 0
- net /Channel0/channel_power/LOAD1_SW_HIGH: track 81.0 -> 0.00 mm, vias 2 -> 0
- net /Channel0/channel_power/LOAD0_SW_HIGH: track 75.4 -> 0.00 mm, vias 2 -> 0
- net /Channel0/T_{TIP}_{a}: track 73.6 -> 0.00 mm, vias 2 -> 0
- net /Channel0/SEL2_{a}: track 66.3 -> 0.00 mm, vias 2 -> 0
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- added copper zone on B.Cu, net /Channel0/channel_meas/CURRENT
- added copper zone on In1.Cu, net GND
- added copper zone on In2.Cu, net GND
- added copper zone on In1.Cu, net Net-(Q801A-S)
- added copper zone on In2.Cu, net Net-(Q801A-S)
- added copper zone on In1.Cu, net Net-(Q802A-S)
- added copper zone on In2.Cu, net Net-(Q802A-S)
- added copper zone on In1.Cu, net Net-(Q803A-S)
- added copper zone on In2.Cu, net Net-(Q803A-S)
- added copper zone on In1.Cu, net Net-(Q807A-S)
- added copper zone on In2.Cu, net Net-(Q807A-S)
- added copper zone on In1.Cu, net Net-(Q808A-S)
- added copper zone on In2.Cu, net Net-(Q808A-S)
Other:
- board size 125 x 60 mm -> 128 x 60 mm
- copper layers 2 -> 4
