File: hardware/SolderOtto/power_latch.kicad_sch (KiCad schematic)
At the start: 4 parts, among them U701 SN74LVC125A, U702 TS5A3159ADCK

Commit message: remove low side switching ic
Parts:
- removed C702: 100n, Capacitor_SMD:C_0603_1608Metric, symbol Device:C
- removed U702: TS5A3159ADCK, Package_TO_SOT_SMD:SOT-363_SC-70-6, symbol Analog_Switch:TS5A3159ADCK
Connections:
- net OUT_COM_L renamed LOW_SIDE_COM
- net OUT_LOAD_L renamed LOW_SIDE_LOAD

Commit message: rework pcb
Connections:
- net IN_LOAD0: now also U701.9 (A); no longer U701.5 (A)
- net IN_LOAD1: now also U701.5 (A); no longer U701.9 (A)
- net OUT_LOAD0_H: now also U701.8 (Y); no longer U701.6 (Y)
- net OUT_LOAD1_H: now also U701.6 (Y); no longer U701.8 (Y)
Other:
- moved on the sheet: U701B, U701C
Changed lines of the file:
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@@
 	(symbol
 		(lib_id "mylib_ic:SN74LVC125A")
-		(at 149.86 101.6 0)
+		(at 149.86 119.38 0)
 		(unit 2)
 		(exclude_from_sim no)
@@
 		(fields_autoplaced yes)
 		(property "Reference" "U701"
-			(at 149.86 92.71 0)
+			(at 149.86 110.49 0)
 			(effects
 				(font
@@
 		)
 		(property "Value" "SN74LVC125A"
-			(at 149.86 95.25 0)
+			(at 149.86 113.03 0)
 			(effects
 				(font
@@
 		)
 		(property "Footprint" "Package_SO:TSSOP-14_4.4x5mm_P0.65mm"
-			(at 149.86 101.6 0)
-			(effects
-				(font
-					(size 1.27 1.27)
-				)
-				(hide yes)
-			)
-		)
-		(property "Datasheet" ""
-			(at 149.86 101.6 0)
+			(at 149.86 119.38 0)
+			(effects
+				(font
+					(size 1.27 1.27)
+				)
+				(hide yes)
+			)
+		)
+		(property "Datasheet" ""
+			(at 149.86 119.38 0)
 			(effects
 				(font
@@
 		)
 		(property "Description" ""
-			(at 149.86 101.6 0)
+			(at 149.86 119.38 0)
 			(effects
 				(font
@@
 		)
 		(property "Digikey" "296-1222-1-ND"
-			(at 149.86 101.6 0)
+			(at 149.86 119.38 0)
 			(effects
 				(font
@@
 	(symbol
 		(lib_id "mylib_ic:SN74LVC125A")
-		(at 149.86 119.38 0)
+		(at 149.86 101.6 0)
 		(unit 3)
 		(exclude_from_sim no)
@@
 		(fields_autoplaced yes)
 		(property "Reference" "U701"
-			(at 149.86 110.49 0)
+			(at 149.86 92.71 0)
 			(effects
 				(font
@@
 		)
 		(property "Value" "SN74LVC125A"
-			(at 149.86 113.03 0)
+			(at 149.86 95.25 0)
 			(effects
 				(font
@@
 		)
 		(property "Footprint" "Package_SO:TSSOP-14_4.4x5mm_P0.65mm"
-			(at 149.86 119.38 0)
-			(effects
-				(font
-					(size 1.27 1.27)
-				)
-				(hide yes)
-			)
-		)
-		(property "Datasheet" ""
-			(at 149.86 119.38 0)
+			(at 149.86 101.6 0)
+			(effects
+				(font
+					(size 1.27 1.27)
+				)
+				(hide yes)
+			)
+		)
+		(property "Datasheet" ""
+			(at 149.86 101.6 0)
 			(effects
 				(font
@@
 		)
 		(property "Description" ""
-			(at 149.86 119.38 0)
+			(at 149.86 101.6 0)
 			(effects
 				(font
@@
 		)
 		(property "Digikey" "296-1222-1-ND"
-			(at 149.86 119.38 0)
-			(effects
-				(font
+			(at 149.86 101.6 0)
+			(effects
+				(font
