File: hardware/SolderOtto/channel.kicad_sch (KiCad schematic)
At the start: 24 parts, among them J601 Conn_01x07, X601 Binder_IP40_07, X602 Binder_IP40_06, X603 Binder_IP40_07, X604 Hirose RPC1-12RB-6P, X605 Binder_IP40_07, X606 Hirose RPC1-12RB-6P

Commit message: save wip
Parts:
- renumbered C602 to C601, C603 to C602, C604 to C603, D604 to D603, D605 to D604, D606 to D605, R603 to R602, R604 to R603, R605 to R604, R606 to R605, R607 to R606
Changed lines of the file:
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@@
 		(dnp no)
 		(fields_autoplaced yes)
-		(property "Reference" "R605"
+		(property "Reference" "R604"
 			(at 265.43 126.9999 0)
 			(effects
@@
 			(project "SolderOtto"
 				(path "/04e99464-bf33-4a4f-8397-d26b5ec904f3/57a4c2b0-a7ab-4dc9-9bcc-6bd7e1b882d1"
-					(reference "R605")
+					(reference "R604")
 					(unit 1)
 				)
@@
 		(dnp no)
 		(fields_autoplaced yes)
-		(property "Reference" "R607"
+		(property "Reference" "R606"
 			(at 255.27 129.5401 90)
 			(effects
@@
 			(project "SolderOtto"
 				(path "/04e99464-bf33-4a4f-8397-d26b5ec904f3/57a4c2b0-a7ab-4dc9-9bcc-6bd7e1b882d1"
-					(reference "R607")
+					(reference "R606")
 					(unit 1)
 				)
@@
 		(dnp no)
 		(fields_autoplaced yes)
-		(property "Reference" "C604"
+		(property "Reference" "C603"
 			(at 266.7 142.2399 0)
 			(effects
@@
 			(project "SolderOtto"
 				(path "/04e99464-bf33-4a4f-8397-d26b5ec904f3/57a4c2b0-a7ab-4dc9-9bcc-6bd7e1b882d1"
-					(reference "C604")
+					(reference "C603")
 					(unit 1)
 				)
@@
 		(on_board yes)
 		(dnp no)
-		(property "Reference" "D605"
+		(property "Reference" "D604"
 			(at 191.008 130.81 90)
 			(effects
@@
 			(project "SolderOtto"
 				(path "/04e99464-bf33-4a4f-8397-d26b5ec904f3/57a4c2b0-a7ab-4dc9-9bcc-6bd7e1b882d1"
-					(reference "D605")
+					(reference "D604")
 					(unit 1)
 				)
@@
 		(dnp no)
 		(fields_autoplaced yes)
-		(property "Reference" "#PWR0602"
+		(property "Reference" "#PWR0601"
 			(at 246.38 80.01 0)
 			(effects
@@
 			(project "SolderOtto"
 				(path "/04e99464-bf33-4a4f-8397-d26b5ec904f3/57a4c2b0-a7ab-4dc9-9bcc-6bd7e1b882d1"
-					(reference "#PWR0602")
+					(reference "#PWR0601")
 					(unit 1)
 				)
@@
 		(dnp no)
 		(fields_autoplaced yes)
-		(property "Reference" "#PWR0603"
+		(property "Reference" "#PWR0602"
 			(at 262.89 80.01 0)
 			(effects
@@
 			(project "SolderOtto"
 				(path "/04e99464-bf33-4a4f-8397-d26b5ec904f3/57a4c2b0-a7ab-4dc9-9bcc-6bd7e1b882d1"
-					(reference "#PWR0603")
+					(reference "#PWR0602")
 					(unit 1)
 				)
@@
 		(dnp no)
 		(fields_autoplaced yes)
-		(property "Reference" "C602"
+		(property "Reference" "C601"
 			(at 266.7 96.5199 0)
 			(effects
@@
 			(project "SolderOtto"
 				(path "/04e99464-bf33-4a4f-8397-d26b5ec904f3/57a4c2b0-a7ab-4dc9-9bcc-6bd7e1b882d1"
-					(reference "C602")
+					(reference "C601")
 					(unit 1)
 				)
@@
 		(on_board yes)
 		(dnp no)
-		(property "Reference" "D606"
+		(property "Reference" "D605"
 			(at 246.888 130.81 90)
 			(effects
@@
 			(project "SolderOtto"
 				(path "/04e99464-bf33-4a4f-8397-d26b5ec904f3/57a4c2b0-a7ab-4dc9-9bcc-6bd7e1b882d1"
-					(reference "D606")
+					(reference "D605")
 					(unit 1)
 				)
@@
 		(dnp no)
 		(fields_autoplaced yes)
-		(property "Reference" "#PWR0613"
+		(property "Reference" "#PWR0610"
 			(at 207.01 156.21 0)
 			(effects
@@
 			(project "SolderOtto"
 				(path "/04e99464-bf33-4a4f-8397-d26b5ec904f3/57a4c2b0-a7ab-4dc9-9bcc-6bd7e1b882d1"
-					(reference "#PWR0613")
+					(reference "#PWR0610")
 					(unit 1)
 				)
@@
 		(dnp no)
 		(fields_autoplaced yes)
-		(property "Reference" "#PWR0606"
+		(property "Reference" "#PWR0603"
 			(at 246.38 110.49 0)
 			(effects
@@
 			(project "SolderOtto"
 				(path "/04e99464-bf33-4a4f-8397-d26b5ec904f3/57a4c2b0-a7ab-4dc9-9bcc-6bd7e1b882d1"
-					(reference "#PWR0606")
+					(reference "#PWR0603")
 					(unit 1)
 				)
@@
 		(dnp no)
 		(fields_autoplaced yes)
-		(property "Reference" "C603"
+		(property "Reference" "C602"
 			(at 210.82 142.2399 0)
 			(effects
@@
 			(project "SolderOtto"
 				(path "/04e99464-bf33-4a4f-8397-d26b5ec904f3/57a4c2b0-a7ab-4dc9-9bcc-6bd7e1b882d1"
-					(reference "C603")
+					(reference "C602")
 					(unit 1)
 				)
@@
 		(on_board yes)
 		(dnp no)
-		(property "Reference" "D604"
+		(property "Reference" "D603"
 			(at 246.888 85.09 90)
 			(effects
@@
 			(project "SolderOtto"
 				(path "/04e99464-bf33-4a4f-8397-d26b5ec904f3/57a4c2b0-a7ab-4dc9-9bcc-6bd7e1b882d1"
-					(reference "D604")
+					(reference "D603")
 					(unit 1)
 				)
@@
 		(dnp no)
 		(fields_autoplaced yes)
-		(property "Reference" "#PWR0609"
+		(property "Reference" "#PWR0606"
 			(at 207.01 125.73 0)
 			(effects
@@
 			(project "SolderOtto"
 				(path "/04e99464-bf33-4a4f-8397-d26b5ec904f3/57a4c2b0-a7ab-4dc9-9bcc-6bd7e1b882d1"
-					(reference "#PWR0609")
+					(reference "#PWR0606")
 					(unit 1)
 				)
@@
 		(dnp no)
 		(fields_autoplaced yes)
-		(property "Reference" "R606"
+		(property "Reference" "R605"
 			(at 199.39 129.54 90)
 			(effects
@@
 			(project "SolderOtto"
 				(path "/04e99464-bf33-4a4f-8397-d26b5ec904f3/57a4c2b0-a7ab-4dc9-9bcc-6bd7e1b882d1"
-					(reference "R606")
+					(reference "R605")
 					(unit 1)
 				)
@@
 		(dnp no)
 		(fields_autoplaced yes)
-		(property "Reference" "#PWR0608"
+		(property "Reference" "#PWR0605"
 			(at 190.5 125.73 0)
 			(effects
@@
 			(project "SolderOtto"
 				(path "/04e99464-bf33-4a4f-8397-d26b5ec904f3/57a4c2b0-a7ab-4dc9-9bcc-6bd7e1b882d1"
-					(reference "#PWR0608")
+					(reference "#PWR0605")
 					(unit 1)
 				)
@@
 		(dnp no)
 		(fields_autoplaced yes)
-		(property "Reference" "R603"
+		(property "Reference" "R602"
 			(at 255.27 83.82 90)
 			(effects
@@
 			(project "SolderOtto"
 				(path "/04e99464-bf33-4a4f-8397-d26b5ec904f3/57a4c2b0-a7ab-4dc9-9bcc-6bd7e1b882d1"
-					(reference "R603")
+					(reference "R602")
 					(unit 1)
 				)
@@
 		(dnp no)
 		(fields_autoplaced yes)
-		(property "Reference" "#PWR0610"
+		(property "Reference" "#PWR0607"
 			(at 246.38 125.73 0)
 			(effects
@@
 			(project "SolderOtto"
 				(path "/04e99464-bf33-4a4f-8397-d26b5ec904f3/57a4c2b0-a7ab-4dc9-9bcc-6bd7e1b882d1"
-					(reference "#PWR0610")
+					(reference "#PWR0607")
 					(unit 1)
 				)
@@
 		(dnp no)
 		(fields_autoplaced yes)
-		(property "Reference" "#PWR0611"
+		(property "Reference" "#PWR0608"
 			(at 262.89 125.73 0)
 			(effects
@@
 			(project "SolderOtto"
 				(path "/04e99464-bf33-4a4f-8397-d26b5ec904f3/57a4c2b0-a7ab-4dc9-9bcc-6bd7e1b882d1"
-					(reference "#PWR0611")
+					(reference "#PWR0608")
 					(unit 1)
 				)
@@
 		(dnp no)
 		(fields_autoplaced yes)
-		(property "Reference" "#PWR0607"
+		(property "Reference" "#PWR0604"
 			(at 262.89 110.49 0)
 			(effects
@@
 			(project "SolderOtto"
 				(path "/04e99464-bf33-4a4f-8397-d26b5ec904f3/57a4c2b0-a7ab-4dc9-9bcc-6bd7e1b882d1"
-					(reference "#PWR0607")
+					(reference "#PWR0604")
 					(unit 1)
 				)
@@
 		(dnp no)
 		(fields_autoplaced yes)
-		(property "Reference" "#PWR0615"
+		(property "Reference" "#PWR0612"
 			(at 262.89 156.21 0)
 			(effects
@@
 			(project "SolderOtto"
 				(path "/04e99464-bf33-4a4f-8397-d26b5ec904f3/57a4c2b0-a7ab-4dc9-9bcc-6bd7e1b882d1"
-					(reference "#PWR0615")
+					(reference "#PWR0612")
 					(unit 1)
 				)
@@
 		(dnp no)
 		(fields_autoplaced yes)
-		(property "Reference" "R604"
+		(property "Reference" "R603"
 			(at 209.55 126.9999 0)
 			(effects
@@
 			(project "SolderOtto"
 				(path "/04e99464-bf33-4a4f-8397-d26b5ec904f3/57a4c2b0-a7ab-4dc9-9bcc-6bd7e1b882d1"
-					(reference "R604")
+					(reference "R603")
 					(unit 1)
 				)
@@
 		(dnp no)
 		(fields_autoplaced yes)
-		(property "Reference" "#PWR0614"
+		(property "Reference" "#PWR0611"
 			(at 246.38 156.21 0)
 			(effects
@@
 			(project "SolderOtto"
 				(path "/04e99464-bf33-4a4f-8397-d26b5ec904f3/57a4c2b0-a7ab-4dc9-9bcc-6bd7e1b882d1"
-					(reference "#PWR0614")
+					(reference "#PWR0611")
 					(unit 1)
 				)
@@
 		(dnp no)
 		(fields_autoplaced yes)
-		(property "Reference" "#PWR0612"
+		(property "Reference" "#PWR0609"
 			(at 190.5 156.21 0)
 			(effects
@@
 			(project "SolderOtto"
 				(path "/04e99464-bf33-4a4f-8397-d26b5ec904f3/57a4c2b0-a7ab-4dc9-9bcc-6bd7e1b882d1"
-					(reference "#PWR0612")
-					(unit 1)
-				)
+					(reference "#PWR0609")
+					(unit 1)
+				)

Commit message: rework schematic foir single channel
Parts:
- added C601, C607, C608, C628: 47p, Capacitor_SMD:C_0603_1608Metric, symbol Device:C
- added C602, C609, C610, C629: 1n, Capacitor_SMD:C_0603_1608Metric, symbol Device:C
- added C603, C606, C611, C614, C615, C616, C617, C618, C619, C620, C621, C622, C623, C624: 100n, Capacitor_SMD:C_0603_1608Metric, symbol Device:C
- added C604, C605, C612, C613: 1u, Capacitor_SMD:C_0603_1608Metric, symbol Device:C
- added D601, D602, D603, D609: BAT54SFILM, Package_TO_SOT_SMD:SOT-23, symbol mylib_diodes:BAT54SFILM
- added F601: 1.25A, Fuse:Fuse_0603_1608Metric, symbol Device:Fuse
- added Q601, Q602: Q_Dual_NMOS, Package_SO:SO-8_3.9x4.9mm_P1.27mm, symbol Device:Q_Dual_NMOS_S1G1S2G2D2D2D1D1
- added Q603, Q604: DTD123EK, Package_TO_SOT_SMD:SC-59, symbol Transistor_BJT:DTD123E
- added R601, R611, R613, R626: 590k, Resistor_SMD:R_0603_1608Metric, symbol Device:R
- added R602, R603, R605, R607, R610, R615, R616, R618, R621, R625: 22k6, Resistor_SMD:R_0603_1608Metric, symbol Device:R
- added R604, R612, R617, R628: 2k7, Resistor_SMD:R_0603_1608Metric, symbol Device:R
- added R606, R619: 2k2, Resistor_SMD:R_0603_1608Metric, symbol Device:R
- added R608, R609: 470, Resistor_SMD:R_0603_1608Metric, symbol Device:R
- added R614, R629: 453k, Resistor_SMD:R_0603_1608Metric, symbol Device:R
- added R620, R624, R639, R641: 3k3, Resistor_SMD:R_0603_1608Metric, symbol Device:R
- added R622, R627: 20k, Resistor_SMD:R_0603_1608Metric, symbol Device:R
- added R623: 5m, Resistor_SMD:R_Shunt_Vishay_WSKW0612, symbol Device:R_Shunt
- added R634, R643: 4k75, Resistor_SMD:R_0603_1608Metric, symbol Device:R
- added R635, R646: 200k, Resistor_SMD:R_0603_1608Metric, symbol Device:R
- added R638, R642: 220m, Resistor_SMD:R_2512_6332Metric, symbol Device:R
- added R640, R647: 10k, Resistor_SMD:R_0603_1608Metric, symbol Device:R
- added R644: 187k, Resistor_SMD:R_0603_1608Metric, symbol Device:R
- added R645: 1M, Resistor_SMD:R_0603_1608Metric, symbol Device:R
- added R648, R649: 10M, Resistor_SMD:R_1206_3216Metric, symbol Device:R
- added TP601, TP602: T_{TIP}, TestPoint:TestPoint_Keystone_5015_Micro-Minature, symbol Connector:TestPoint
- added TP603: I_{LOAD}, TestPoint:TestPoint_Keystone_5015_Micro-Minature, symbol Connector:TestPoint
- added TP604: I_{LEAK}, TestPoint:TestPoint_Keystone_5015_Micro-Minature, symbol Connector:TestPoint
- added U601, U606, U607: OPA202, Package_SO:SOIC-8_3.9x4.9mm_P1.27mm, symbol mylib_ic:OPA206
- added U602: LM358B, Package_SO:SOIC-8_3.9x4.9mm_P1.27mm, symbol Amplifier_Operational:LM358
- added U603, U608: TMUX4053, Package_SO:TSSOP-16_4.4x5mm_P0.65mm, symbol mylib_ic:TMUX4053
- added U604, U605: VOM1271, mylib_ic:SOP-4_3.8x4.1mm_P2.54mm, symbol mylib_diodes:VOM1271
- added U609: OPA2186, Package_SO:SOIC-8_3.9x4.9mm_P1.27mm, symbol Amplifier_Operational:OPA2196xD
- renumbered C601 to C625, C602 to C626, C603 to C627, D603 to D604, D601 to D605, D602 to D606, D604 to D607, D605 to D608, HEATER603 to HEATER602, HEATER602 to HEATER603, R601 to R630, R602 to R631, R603 to R632, R604 to R633, R605 to R636, R606 to R637, X605 to X603, X606 to X604, X603 to X605, X604 to X606
Connections:
- net +3V3: now also D601.2, D602.2, D603.2, D609.2, R620.1, R639.1
- net COM: now also R603.1, R616.1, R623.1
- net GND: now also C602.2, C603.2, C604.2, C605.2, C606.2, C609.2, C610.2, C611.2, C612.2, C613.2, C614.2, C615.2, C616.2, C617.2, C618.2, C619.1, C620.2, C621.2, C622.2, C623.2, C624.2, C629.2, D601.1, D602.1, D603.1, D609.1, Q603.2 (E), Q604.2 (E), R611.2, R612.2, R623.4, R626.2, R628.2, R629.1, R646.1, R647.1, U603.6 (~{E}), U603.8 (GND), U608.6 (~{E}), U608.8 (GND)
- net I_{LEAK}: now also C629.1, D609.3, R639.2, R641.1, TP604.1
- net I_{LOAD}: now also C610.1, D603.3, R620.2, R624.1, TP603.1
- net LOAD0_SW: now also Q604.1 (B)
- net LOAD1_SW: now also Q603.1 (B)
- net SEL1_{a}: now also U603.9 (S1)
- net SEL1_{b}: now also U608.9 (S1)
- net SEL2_{a}: now also U603.10 (S2)
- net SEL2_{b}: now also U608.10 (S2)
- net TC: now also R602.1, R607.1, R615.1, R621.1, R634.1, R638.1
- net T_{TIP}_{a}: now also C602.1, D601.3, R606.2, TP601.1
- net T_{TIP}_{b}: now also C609.1, D602.3, R619.2, TP602.1
- new net: R610.1, R612.1, U602.6 (-)
- new net: R622.1, R623.2
- new net: R623.3, R627.1
- new net: R605.2, U603.2 (S2A)
- new net: F601.1, R642.2, R643.2, R645.1
- new net: R621.2, U608.1 (S2B)
- new net: Q602.1 (S), Q602.3 (S), U605.3
- new net: Q602.2 (G), Q602.4 (G), U605.4
- new net: C628.1, R634.2, R635.1, U609.2 (-)
- new net: C628.2, R643.1, R646.2, U609.3 (+)
- new net: R635.2, R640.1, U609.1
- new net: C601.2, R611.1, U601.3 (+), U603.15 (D2)
- new net: R609.2, U605.1
- new net: Q604.3 (C), U605.2
- new net: R641.2, R644.2, U609.7
- new net: C607.2, R626.1, U606.3 (+), U608.15 (D2)
- new net: R618.2, U608.2 (S2A)
- new net: R616.2, U608.3 (S1B)
- new net: C607.1, R613.1, U606.2 (-), U608.4 (D1)
- new net: R615.2, U608.5 (S1A)
- new net: C608.2, R627.2, R629.2, U607.3 (+)
- new net: Q601.1 (S), Q601.3 (S), U604.3
- new net: Q601.2 (G), Q601.4 (G), U604.4
- new net: R644.1, R647.2, U609.6 (-)
- new net: Q603.3 (C), U604.2
- new net: U601.1 (NC), U601.5 (NC), U601.8 (NC)
- new net: C601.1, R601.1, U601.2 (-), U603.4 (D1)
- new net: R601.2, R604.1, U601.6
- new net: R613.2, R617.1, U606.6
- new net: R617.2, U602.3 (+)
- new net: R604.2, U602.5 (+)
- new net: R638.2, R642.1
- new net: R614.2, R624.2, U607.6
- new net: R640.2, U609.5 (+)
- new net: R619.1, R625.2, U602.1
- new net: R625.1, R628.1, U602.2 (-)
- new net: R603.2, U603.3 (S1B)
- new net: C608.1, R614.1, R622.2, U607.2 (-)
- new net: R606.1, R610.2, U602.7
- new net: R602.2, U603.5 (S1A)
- new net: R608.2, U604.1
- new net: R607.2, U603.1 (S2B)
- new net: U607.1 (NC), U607.5 (NC), U607.8 (NC)
- new net: U606.1 (NC), U606.5 (NC), U606.8 (NC)
- new net +5V: C603.1, C604.1, C611.1, C612.1, U603.16 (VCC), U608.16 (VCC)
- new net +8V: C615.1, C616.1, C617.1, C618.1, C619.2, R608.1, R609.1, U601.7 (V+), U602.8 (V+), U606.7 (V+), U607.7 (V+), U609.8 (V+)
- new net -5V: C605.1, C606.1, C613.1, C614.1, C620.1, C621.1, C622.1, C623.1, C624.1, U601.4 (V-), U602.4 (V-), U603.7 (VEE), U606.4 (V-), U607.4 (V-), U608.7 (VEE), U609.4 (V-)
- new net 24V_{AC}: Q601.7 (D), Q601.8 (D), Q602.7 (D), Q602.8 (D), R648.1, R649.1
- new net Earth: F601.2, R645.2
- new net LOAD0: Q602.5 (D), Q602.6 (D), R605.1, R649.2
- new net LOAD1: Q601.5 (D), Q601.6 (D), R618.1, R648.2
- no-connect marks 8 -> 16
Other:
- removed sheet channel_meas
- removed sheet channel_power
- moved on the sheet: C625, C626, C627, D604, D607, D608, J601, R630, R631, R632, R633, R636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
