File: hardware/SolderOtto/channel.kicad_sch (KiCad schematic)
At the start: 126 parts, among them J601 Conn_01x07, J602 Conn_01x07, Q601 Q_Dual_NMOS, Q602 Q_Dual_NMOS, Q603 DTD123EK, Q604 DTD123EK, Q605 BC847A, Q606 BC858B, Q607 BC847A, U601 OPA2186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

Commit message: update some shit
Parts:
- C611: Digikey (none) -> 1276-1008-1-ND
- R610, R611: Digikey (none) -> 311-10.0MFRCT-ND
- R624: Digikey (none) -> 311-470KHRCT-ND
- R626, R632: Digikey (none) -> 311-47.0KHRCT-ND
- R640, R649: Digikey (none) -> P4.75KHCT-ND
- R641, R652: Digikey (none) -> 311-200KHRCT-ND
- R650: Digikey (none) -> P187KHCT-ND
- U601, U605, U608: Digikey (none) -> 296-OPA2186DRCT-ND
Changed lines of the file:
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@@
 			)
 		)
+		(property "Digikey" "296-OPA2186DRCT-ND"
+			(at 318.77 40.64 0)
+			(effects
+				(font
+					(size 1.27 1.27)
+				)
+				(hide yes)
+			)
+		)
 		(pin "3"
 		)
@@
 			)
 		)
-		(property "Digikey" ""
+		(property "Digikey" "311-47.0KHRCT-ND"
 			(at 165.1 120.65 0)
 			(effects
@@
 			)
 		)
-		(property "Digikey" ""
+		(property "Digikey" "P4.75KHCT-ND"
 			(at 157.48 224.79 0)
 			(effects
@@
 			)
 		)
-		(property "Digikey" ""
+		(property "Digikey" "P4.75KHCT-ND"
 			(at 157.48 247.65 0)
 			(effects
@@
 			)
 		)
+		(property "Digikey" "296-OPA2186DRCT-ND"
+			(at 351.79 43.18 0)
+			(effects
+				(font
+					(size 1.27 1.27)
+				)
+				(hide yes)
+			)
+		)
 		(pin "3"
 		)
@@
 			)
 		)
-		(property "Digikey" ""
+		(property "Digikey" "311-200KHRCT-ND"
 			(at 181.61 224.79 0)
 			(effects
@@
 			)
 		)
-		(property "Digikey" ""
+		(property "Digikey" "311-47.0KHRCT-ND"
 			(at 205.74 113.03 0)
 			(effects
@@
 			)
 		)
+		(property "Digikey" "296-OPA2186DRCT-ND"
+			(at 181.61 236.22 0)
+			(effects
+				(font
+					(size 1.27 1.27)
+				)
+				(hide yes)
+			)
+		)
 		(pin "3"
 		)
@@
 			)
 		)
+		(property "Digikey" "296-OPA2186DRCT-ND"
+			(at 213.36 238.76 0)
+			(effects
+				(font
+					(size 1.27 1.27)
+				)
+				(hide yes)
+			)
+		)
 		(pin "3"
 		)
@@
 			)
 		)
+		(property "Digikey" "296-OPA2186DRCT-ND"
+			(at 158.75 175.26 0)
+			(effects
+				(font
+					(size 1.27 1.27)
+				)
+				(hide yes)
+			)
+		)
 		(pin "3"
 		)
@@
 			)
 		)
-		(property "Digikey" ""
+		(property "Digikey" "311-10.0MFRCT-ND"
 			(at 100.33 52.07 0)
 			(effects
@@
 			)
 		)
+		(property "Digikey" "296-OPA2186DRCT-ND"
+			(at 351.79 107.95 0)
+			(effects
+				(font
+					(size 1.27 1.27)
+				)
+				(hide yes)
+			)
+		)
 		(pin "3"
 		)
@@
 			)
 		)
-		(property "Digikey" ""
+		(property "Digikey" "311-200KHRCT-ND"
 			(at 172.72 256.54 0)
 			(effects
@@
 			)
 		)
-		(property "Digikey" ""
+		(property "Digikey" "P187KHCT-ND"
 			(at 214.63 250.19 0)
 			(effects
@@
 			)
 		)
-		(property "Digikey" ""
+		(property "Digikey" "311-10.0MFRCT-ND"
 			(at 194.31 52.07 0)
 			(effects
@@
 			)
 		)
-		(property "Digikey" ""
+		(property "Digikey" "1276-1008-1-ND"
 			(at 175.26 128.27 0)
 			(effects
@@
 			)
 		)
+		(property "Digikey" "296-OPA2186DRCT-ND"
+			(at 134.62 175.26 0)
+			(effects
+				(font
+					(size 1.27 1.27)
+				)
+				(hide yes)
+			)
+		)
 		(pin "3"
 		)
@@
 			)
 		)
+		(property "Digikey" "296-OPA2186DRCT-ND"
+			(at 209.55 175.26 0)
+			(effects
+				(font
+					(size 1.27 1.27)
+				)
+				(hide yes)
+			)
+		)
 		(pin "3"
 		)
@@
 			)
 		)
-		(property "Digikey" ""
+		(property "Digikey" "311-470KHRCT-ND"
 			(at 160.02 111.76 0)
 			(effects
@@
 			(at 318.77 105.41 0)
 			(effects
+				(font
+					(size 1.27 1.27)
+				)
+				(hide yes)
+			)
+		)
+		(property "Digikey" "296-OPA2186DRCT-ND"
+			(at 318.77 105.41 0)
+			(effects
