File: hardware/SolderOtto/display.kicad_sch (KiCad schematic)
At the start: 1 part, among them J401 Conn_01x20

Commit message: save wip
Connections:
- net QSPI_IO0 renamed SPI_MOSI
- net QSPI_IO1 renamed SPI_MISO
Changed lines of the file:
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@@
 	(wire
 		(pts
-			(xy 151.13 63.5) (xy 151.13 71.12)
+			(xy 138.43 53.34) (xy 138.43 63.5)
 		)
 		(stroke
@@
 	(wire
 		(pts
+			(xy 138.43 63.5) (xy 129.54 63.5)
+		)
+		(stroke
+			(width 0)
+			(type default)
+		)
+	)
+	(wire
+		(pts
+			(xy 138.43 53.34) (xy 142.24 53.34)
+		)
+		(stroke
+			(width 0)
+			(type default)
+		)
+	)
+	(wire
+		(pts
 			(xy 137.16 78.74) (xy 129.54 78.74)
 		)
@@
 	(wire
 		(pts
+			(xy 129.54 71.12) (xy 137.16 71.12)
+		)
+		(stroke
+			(width 0)
+			(type default)
+		)
+	)
+	(wire
+		(pts
 			(xy 134.62 114.3) (xy 134.62 109.22)
 		)
@@
 	(wire
 		(pts
-			(xy 129.54 63.5) (xy 151.13 63.5)
+			(xy 129.54 68.58) (xy 137.16 68.58)
 		)
 		(stroke
@@
 	(wire
 		(pts
-			(xy 137.16 71.12) (xy 129.54 71.12)
+			(xy 142.24 53.34) (xy 142.24 54.61)
 		)
 		(stroke
@@
 		(pts
 			(xy 137.16 66.04) (xy 129.54 66.04)
-		)
-		(stroke
-			(width 0)
-			(type default)
-		)
-	)
-	(wire
-		(pts
-			(xy 137.16 68.58) (xy 129.54 68.58)
 		)
 		(stroke
@@
 		)
 	)
-	(hierarchical_label "QSPI_IO1"
-		(shape bidirectional)
-		(at 137.16 68.58 0)
-		(fields_autoplaced yes)
-		(effects
-			(font
-				(size 1.27 1.27)
-			)
-			(justify left)
-		)
-	)
 	(hierarchical_label "QSPI_CS"
 		(shape input)
@@
 		)
 	)
-	(hierarchical_label "QSPI_IO0"
-		(shape bidirectional)
-		(at 137.16 71.12 0)
-		(fields_autoplaced yes)
-		(effects
-			(font
-				(size 1.27 1.27)
-			)
-			(justify left)
-		)
-	)
 	(hierarchical_label "~{INT}"
 		(shape output)
@@
 		)
 	)
+	(hierarchical_label "SPI_MISO"
+		(shape bidirectional)
+		(at 137.16 68.58 0)
+		(fields_autoplaced yes)
+		(effects
+			(font
+				(size 1.27 1.27)
+			)
+			(justify left)
+		)
+	)
 	(hierarchical_label "AUDIO_OUT"
 		(shape output)
@@
 		(shape bidirectional)
 		(at 137.16 86.36 0)
+		(fields_autoplaced yes)
+		(effects
+			(font
+				(size 1.27 1.27)
+			)
+			(justify left)
+		)
+	)
+	(hierarchical_label "SPI_MOSI"
+		(shape bidirectional)
+		(at 137.16 71.12 0)
 		(fields_autoplaced yes)
 		(effects
@@
 	(symbol
 		(lib_id "power:GND")
-		(at 151.13 71.12 0)
+		(at 142.24 54.61 0)
 		(unit 1)
 		(exclude_from_sim no)
@@
 		(fields_autoplaced yes)
 		(property "Reference" "#PWR0402"
-			(at 151.13 77.47 0)
+			(at 142.24 60.96 0)
 			(effects
 				(font
@@
 		)
 		(property "Value" "GND"
-			(at 151.13 76.2 0)
+			(at 142.24 59.69 0)
 			(effects
 				(font
@@
 		)
 		(property "Footprint" ""
-			(at 151.13 71.12 0)
+			(at 142.24 54.61 0)
 			(effects
 				(font
@@
 		)
 		(property "Datasheet" ""
-			(at 151.13 71.12 0)
+			(at 142.24 54.61 0)
 			(effects
 				(font
@@
 		)
 		(property "Description" "Power symbol creates a global label with name \"GND\" , ground"
-			(at 151.13 71.12 0)
-			(effects
-				(font
+			(at 142.24 54.61 0)
+			(effects
+				(font
