File: hardware/SolderOtto/mcu.kicad_sch (KiCad schematic)
At the start: 24 parts, among them J302 Conn_ARM_SWD_TagConnect_TC2030, P301 USB_C_Plug_USB2.0, SW301 SW_Push, U301 USBLC6-2SC6, U302 STM32G474RETx, U303 MX25R3235FM1xx0, Y301 32.768 kHz

Commit message: update some shit
Parts:
- P301: Digikey (none) -> 900-2171790001CT-ND
- U302: Digikey (none) -> 497-STM32G474RET6-ND
Changed lines of the file:
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@@
+			)
+		)
+		(property "Digikey" "497-STM32G474RET6-ND"
+			(at 187.96 144.78 0)
+			(effects
+				(font
+					(size 1.27 1.27)
+				)
 			)
 		)
@@
 			)
 		)
-		(property "Digikey" ""
+		(property "Digikey" "900-2171790001CT-ND"
 			(at 43.18 77.47 0)
 			(effects
