File: cad/hardware/SolderOtto/mcu.kicad_sch (KiCad schematic)
At the start: 24 parts, among them J302 Conn_ARM_SWD_TagConnect_TC2030, P301 USB_C_Plug_USB2.0, SW301 SW_Push, U301 USBLC6-2SC6, U302 STM32G474RETx, U303 MX25R3235FM1xx0, Y301 32.768 kHz

Commit message: Implements basic ADC and display functionality
This commit sets up the basic application framework.

It adds wave control initialization, display functionality using BT81x, and ADC configurations for voltage and temperature measurements.
Also, it adds include directories and source files to CMakeLists, as well as fixes git ignore and device tree configurations.
The removal of the previous main.c and addition of separate c files allows for better modularity and organization.
Connections:
- net QSPI_CLK: now also U303.6 (SCLK); no longer U303.1 (~{CS})
- net QSPI_NCS: now also U303.1 (~{CS}); no longer U303.6 (SCLK)
Changed lines of the file:
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@@
 	)
 	(label "QSPI_NCS"
-		(at 67.31 156.21 180)
+		(at 67.31 153.67 180)
 		(effects
 			(font
@@
 	)
 	(label "QSPI_CLK"
-		(at 67.31 153.67 180)
+		(at 67.31 156.21 180)
 		(effects
 			(font
